File: CS30/ONI-Kyan MKI.kicad_pcb (KiCad board)
At the start: 2 copper layers, 239.8 x 99.7 mm, 69 parts, among them U0 ProMicro

Commit message: Finalized ONI-Kyan MK-I
Created gerbers and ordered prototypes through JLCPCB
Parts:
- SS0: renamed from G***; value LOGO -> MKII SS
- SS1: renamed from G***; value LOGO -> ONI-Kyan Logo Front
- SS2: renamed from G***; value LOGO -> ONI-Kyan Logo Back
Changed lines of the file:
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@@
   (module OniKyan-SS:MkII (layer F.Cu)
     (at 142.8756 110)
-    (fp_text reference G*** (at 0 0) (layer F.SilkS) hide
+    (fp_text reference SS0 (at 0 0) (layer F.SilkS) hide
       (effects (font (size 1.524 1.524) (thickness 0.3)))
     )
-    (fp_text value LOGO (at 0.75 0) (layer F.SilkS) hide
+    (fp_text value "MKII SS" (at 0.75 0) (layer F.SilkS) hide
       (effects (font (size 1.524 1.524) (thickness 0.3)))
     )
@@
   (module OniKyan-SS:OniKyan_SS (layer F.Cu)
     (at 141.5 130.825519)
-    (fp_text reference G*** (at 0 0) (layer F.SilkS) hide
+    (fp_text reference SS1 (at 0 0) (layer F.SilkS) hide
       (effects (font (size 1.524 1.524) (thickness 0.3)))
     )
-    (fp_text value LOGO (at 0.75 0) (layer F.SilkS) hide
+    (fp_text value "ONI-Kyan Logo Front" (at 0.75 0) (layer F.SilkS) hide
       (effects (font (size 1.524 1.524) (thickness 0.3)))
     )
@@
   (module OniKyan-SS:OniKyan_SS (layer B.Cu)
     (at 144.600001 130.825519 180)
-    (fp_text reference G*** (at 0 0) (layer B.SilkS) hide
+    (fp_text reference SS2 (at 0 0) (layer B.SilkS) hide
       (effects (font (size 1.524 1.524) (thickness 0.3)) (justify mirror))
     )
-    (fp_text value LOGO (at 0.75 0) (layer B.SilkS) hide
+    (fp_text value "ONI-Kyan Logo Back" (at 0.75 0) (layer B.SilkS) hide
       (effects (font (size 1.524 1.524) (thickness 0.3)) (justify mirror))
     )
